Commit message: feat: add sim-real teleop and assembly experiment foundation

File: assets/robots/linker_platform/combined_robot/lkls73_o2_dual_arm_description.urdf (robot description, URDF)
Before this commit: robot lkls73_o2_dual_arm_description, 17 links, 16 joints
Links:
- added link world
Joints:
- added joint World_Base_Mount_Joint: type fixed, parent world, child Body_Base_link, origin xyz=0 0 -1.052 rpy=0 0 0
- joint Left_Shoulder_Base_Joint: origin xyz=-0.023 0 0 rpy=0 0 0 -> xyz=-0.023 0 1.052 rpy=0 0 0
- joint Right_Shoulder_Base_Joint: origin xyz=-0.023 0 0 rpy=0 0 0 -> xyz=-0.023 0 1.052 rpy=0 0 0
